Commit message: added node to take angles in degress and publish it for FWD script

File: src/robotics/urdf/robot.urdf (robot description, URDF)
Before this commit: robot R5_DOF_Robot_Assembly, 8 links, 7 joints
Joints:
- joint Base_Link_to_world: origin xyz=0 0 0 rpy=0 0 0 -> xyz=0 0 0.050 rpy=0 0 0

Commit message: Milestone_2 update

File: src/robotics/urdf/robot.urdf (robot description, URDF)
Before this commit: robot R5_DOF_Robot_Assembly, 8 links, 7 joints
Links:
- removed link Arm_1
- removed link Arm_2
- removed link Arm_3
- removed link Base_Link
- removed link Gripper
- removed link Rotating_Waste
- added link base_link, mass 0.12603; collision mesh filename=package://robotics/meshes/base_link.STL; visual mesh filename=package://robotics/meshes/base_link.STL
- added link joint1, mass 0.1236; collision mesh filename=package://robotics/meshes/joint1.STL; visual mesh filename=package://robotics/meshes/joint1.STL
- added link joint2, mass 0.13798; collision mesh filename=package://robotics/meshes/joint2.STL; visual mesh filename=package://robotics/meshes/joint2.STL
- added link joint3, mass 0.14179; collision mesh filename=package://robotics/meshes/joint3.STL; visual mesh filename=package://robotics/meshes/joint3.STL
- added link joint4, mass 0.01872; collision mesh filename=package://robotics/meshes/joint4.STL; visual mesh filename=package://robotics/meshes/joint4.STL
- added link joint5, mass 0.04918; collision mesh filename=package://robotics/meshes/joint5.STL; visual mesh filename=package://robotics/meshes/joint5.STL
Joints:
- removed joint Base_Link_to_world
- added joint base_link_to_world: type fixed, parent world, child base_link, origin xyz=0 0 0 rpy=-1.5708 0 0
- joint EE_frame_lock: origin xyz=0.007 0.1 0.013 rpy=0 0 0 -> xyz=0.09 0.0 0.0 rpy=0 0 0; parent Gripper -> joint5
- joint Joint_1: axis 0 0 1 -> 0 1 0; child Rotating_Waste -> joint1; origin xyz=0 0 0 rpy=0 0 0 -> xyz=0.042627 -0.088458 0.04544 rpy=0 -1.5708 3.14159; parent Base_Link -> base_link
- joint Joint_2: axis 0 0 1 -> 0 1 0; child Arm_1 -> joint2; origin xyz=-2.7567E-05 0.0061999 0.04975 rpy=1.5708 0 0 -> xyz=0 0.04355 0 rpy=1.5708 0 1.6019; parent Rotating_Waste -> joint1
- joint Joint_3: axis 0 0 -1 -> 0 0 1; child Arm_2 -> joint3; origin xyz=0 0.140 0.000 rpy=0 0 1.5708 -> xyz=0.14 0 0 rpy=1.5708 -0.031075 0; parent Arm_1 -> joint2
- joint Joint_4: axis 0 0 -1 -> 0 0 1; child Arm_3 -> joint4; origin xyz=0 0 0 rpy=-1.5708 0 -1.5708 -> xyz=0.1329 0.0005 0 rpy=0 0 0; parent Arm_2 -> joint3
- joint Joint_5: axis 0 0 1 -> 1 0 0; child Gripper -> joint5; origin xyz=-0.001651 -0.0054574 0.13289 rpy=1.5708 0 0 -> xyz=0.02245 -0.00038473 -0.0018312 rpy=1.5708 0 0; parent Arm_3 -> joint4

Commit message: Replaced trajectory controller with forward command

File: src/robotics/urdf/robot.urdf (robot description, URDF)
Before this commit: robot New Robot Assmembly.SLDASM, 8 links, 7 joints
Links:
- removed link EE_frame
- removed link joint1
- removed link joint2
- removed link joint3
- removed link joint4
- removed link joint5
- added link arm, mass 0.137984699871301; collision mesh filename=package://robotics/meshes/arm.STL; visual mesh filename=package://robotics/meshes/arm.STL
- added link end_effector, mass 0.04918; collision mesh filename=package://robotics/meshes/end_effector.STL; visual mesh filename=package://robotics/meshes/end_effector.STL
- added link forearm, mass 0.141790967611344; collision mesh filename=package://robotics/meshes/forearm.STL; visual mesh filename=package://robotics/meshes/forearm.STL
- added link rotating_waist, mass 0.123597949087119; collision mesh filename=package://robotics/meshes/rotating_waist.STL; visual mesh filename=package://robotics/meshes/rotating_waist.STL
- added link wrist, mass 0.01872; collision mesh filename=package://robotics/meshes/wrist.STL; visual mesh filename=package://robotics/meshes/wrist.STL
- link base_link: mass 0.12603 -> 0.126025187508608
Joints:
- removed joint EE_frame_lock
- removed joint Joint_1
- removed joint Joint_2
- removed joint Joint_3
- removed joint Joint_4
- removed joint Joint_5
- added joint arm_joint: type revolute, parent rotating_waist, child arm, origin xyz=0.004 0 0.04105 rpy=0 -1.5708 3.14, axis 0 0 1, limit lower=-3.14 upper=3.14 effort=5 velocity=2
- added joint end_effector_joint: type revolute, parent wrist, child end_effector, origin xyz=0.0523 0  -0.0052 rpy=0 1.5708 0, axis 0 0 1, limit lower=-3.14 upper=3.14 effort=5 velocity=2
- added joint forearm_joint: type revolute, parent arm, child forearm, origin xyz=0.13993 0.0043497 0, axis 0 0 -1, limit lower=-3.14 upper=3.14 effort=5 velocity=2
- added joint rotating_waist_joint: type revolute, parent base_link, child rotating_waist, origin xyz=0 0 0.0525, axis 0 0 1, limit lower=-3.14 upper=3.14 effort=5 velocity=2
- added joint wrist_joint: type revolute, parent forearm, child wrist, origin xyz=0.1329 -0.0005 0.00305, axis 0 0 -1, limit lower=-3.14 upper=3.14 effort=5 velocity=2
- joint base_link_to_world: origin xyz=0 0 0 rpy=-1.5708 0 0 -> xyz=0 0 0 rpy=0 0 0
